Commit message: added ultrasound sensors

File: omnirob_robin_description/robots/omnirob_robin_simulated.urdf.xacro (robot description, xacro)
@@ -13,4 +13,28 @@
     <insert_block name="pan_tilt_origin" />
   </xacro:schunk_pan_tilt>
+  <xacro:ultrasound_sensor parent="base_link" number="0">
+    <insert_block name="ultrasound_sensor0" />
+  </xacro:ultrasound_sensor>
+  <xacro:ultrasound_sensor parent="base_link" number="1">
+    <insert_block name="ultrasound_sensor1" />
+  </xacro:ultrasound_sensor>
+  <xacro:ultrasound_sensor parent="base_link" number="2">
+    <insert_block name="ultrasound_sensor2" />
+  </xacro:ultrasound_sensor>
+  <xacro:ultrasound_sensor parent="base_link" number="3">
+    <insert_block name="ultrasound_sensor3" />
+  </xacro:ultrasound_sensor>
+  <xacro:ultrasound_sensor parent="base_link" number="4">
+    <insert_block name="ultrasound_sensor4" />
+  </xacro:ultrasound_sensor>
+  <xacro:ultrasound_sensor parent="base_link" number="5">
+    <insert_block name="ultrasound_sensor5" />
+  </xacro:ultrasound_sensor>
+  <xacro:ultrasound_sensor parent="base_link" number="6">
+    <insert_block name="ultrasound_sensor6" />
+  </xacro:ultrasound_sensor>
+  <xacro:ultrasound_sensor parent="base_link" number="7">
+    <insert_block name="ultrasound_sensor7" />
+  </xacro:ultrasound_sensor>
   <xacro:sensor_kinect parent="pan_tilt/tcp_link" />
   <xacro:sensor_sick3000 parent="base_link" />

File: omnirob_robin_description/urdf/omnirob_robin.library.xacro (robot description, xacro)
@@ -25,3 +25,4 @@
   <xacro:include filename="$(find omnirob_robin_description)/urdf/sensors/kinect2.urdf.xacro"/>
   <xacro:include filename="$(find omnirob_robin_description)/urdf/sensors/sick3000.urdf.xacro"/>
+  <xacro:include filename="$(find omnirob_robin_description)/urdf/sensors/Ultrasound.urdf.xacro"/>
 </robot>

File: omnirob_robin_description/urdf/omnirob_robin.properties.xacro (robot description, xacro)
@@ -41,3 +41,30 @@
     <origin xyz="${0.7/2.0+0.003+0.0597} 0 ${0.293+0.116}" rpy="${M_PI} 0 0"/>
   </xacro:property>
+  <property name="ultrasound_z" value="0.66"/>
+  <property name="ultrasound_offset" value="0.34"/>
+  <property name="sqrt2" value="1.414213562"/>
+  <xacro:property name="ultrasound_sensor0">
+    <origin xyz="${ultrasound_offset} 0.0 ${ultrasound_z}" rpy="0 0 0"/>
+  </xacro:property>
+  <xacro:property name="ultrasound_sensor1">
+    <origin xyz="${ultrasound_offset*1/sqrt2} ${ultrasound_offset*1/sqrt2} ${ultrasound_z}" rpy="0 0 ${M_PI/4}"/>
+  </xacro:property>
+  <xacro:property name="ultrasound_sensor2">
+    <origin xyz="0.0 ${ultrasound_offset} ${ultrasound_z}" rpy="0 0 ${M_PI/2}"/>
+  </xacro:property>
+  <xacro:property name="ultrasound_sensor3">
+    <origin xyz="${ultrasound_offset*1/sqrt2*(-1)} ${ultrasound_offset*1/sqrt2} ${ultrasound_z}" rpy="0 0 ${3*M_PI/4}"/>
+  </xacro:property>
+  <xacro:property name="ultrasound_sensor4">
+    <origin xyz="${ultrasound_offset*(-1)} 0.0 ${ultrasound_z+0.025}" rpy="0 0 ${M_PI}"/>
+  </xacro:property>
+  <xacro:property name="ultrasound_sensor5">
+    <origin xyz="${ultrasound_offset*1/sqrt2*(-1)} ${ultrasound_offset*1/sqrt2*(-1)} ${ultrasound_z}" rpy="0 0 ${5*M_PI/4}"/>
+  </xacro:property>
+  <xacro:property name="ultrasound_sensor6">
+    <origin xyz="0.0 ${ultrasound_offset*(-1)} ${ultrasound_z}" rpy="0 0 ${6*M_PI/4}"/>
+  </xacro:property>
+  <xacro:property name="ultrasound_sensor7">
+    <origin xyz="${ultrasound_offset*1/sqrt2} ${ultrasound_offset*1/sqrt2*(-1)} ${ultrasound_z}" rpy="0 0 ${7*M_PI/4}"/>
+  </xacro:property>
 </robot>
