Commit message: Updated urdfs to work with rospy urd parsers

File: omnirob_robin_description/robots/omnirob.urdf.xacro (robot description, xacro)
@@ -2,5 +2,5 @@
 <robot name="omnirob_robin" xmlns:xacro="http://ros.org/wiki/xacro">
   <xacro:include filename="$(find omnirob_robin_description)/urdf/omnirob_robin.library.xacro" />
-  <!-- load the base of the robot -->
+  <!-- load the base of the robot   -->
   <xacro:base />
   <xacro:camera_mast parent="base_link">

File: omnirob_robin_description/urdf/lwa/lwa.urdf.xacro (robot description, xacro)
@@ -97,5 +97,5 @@
       <axis xyz="0 0 1"/>
       <dynamics damping="0.5" friction="1.0" />
-      <calibration rising="${arm_3_ref}"/>
+      <calibration rising="${arm_3_ref}" falling="0.0"/>
       <limit effort="300" velocity="2.0" lower="-3.14" upper="3.14"/>
       <safety_controller k_position="20" k_velocity="25" soft_lower_limit="${-3.14 + 0.1}" soft_upper_limit="${3.14 - 0.1}" />
@@ -128,5 +128,5 @@
       <axis xyz="0 0 1" />
       <dynamics damping="0.5" friction="1.0" />
-      <calibration rising="${arm_4_ref}"/>
+      <calibration rising="${arm_4_ref}" falling="0.0"/>
       <limit effort="300" velocity="2.0" lower="-2.44" upper="2.44"/>
       <safety_controller k_position="20" k_velocity="25" soft_lower_limit="${-2.44 + 0.01}" soft_upper_limit="${2.44 - 0.01}" />
@@ -159,5 +159,5 @@
       <axis xyz="0 0 1" />
      <dynamics damping="0.5" friction="1.0" />
-      <calibration rising="${arm_5_ref}"/>
+      <calibration rising="${arm_5_ref}" falling="0.0"/>
       <limit effort="300"  velocity="2.0" lower="-3" upper="3" />
       <safety_controller k_position="20" k_velocity="25" soft_lower_limit="${-3 + 0.01}" soft_upper_limit="${3 - 0.01}" />
@@ -190,5 +190,5 @@
       <axis xyz="0 0 1" />
       <dynamics damping="0.5" friction="1.0" />
-      <calibration rising="${arm_6_ref}"/>
+      <calibration rising="${arm_6_ref}" falling="0.0"/>
       <limit effort="300" velocity="2.0" lower="-2.44" upper="2.44" />
       <safety_controller k_position="20" k_velocity="25" soft_lower_limit="${-2.44 + 0.01}" soft_upper_limit="${2.44 - 0.01}" />
@@ -221,5 +221,5 @@
       <axis xyz="0 0 1" />
       <dynamics damping="0.5" friction="1.0" />
-      <calibration rising="${arm_7_ref}"/>
+      <calibration rising="${arm_7_ref}" falling="0.0"/>
       <limit effort="100" velocity="2.0" lower="-3" upper="3" />
       <safety_controller k_position="20" k_velocity="25" soft_lower_limit="${-3 + 0.01}" soft_upper_limit="${3 - 0.01}" />

File: omnirob_robin_description/urdf/omnirob_robin_base/base.urdf.xacro (robot description, xacro)
@@ -1,98 +1,94 @@
-<?xml version="1.0"?>
+<?xml version="1.0" encoding="UTF-8"?>
 <robot xmlns:xacro="http://ros.org/wiki/xacro">
-	<!-- Including Gazebo extensions -->
-	<xacro:include filename="$(find omnirob_robin_description)/urdf/omnirob_robin_base/base.transmission.xacro"/>
-	<xacro:macro name="base" params="">
-    <link name="world" />
-    <joint name="odom_joint" type="fixed">
-			<parent link="world"/>
-			<child link="odom" />
-		</joint>
-    <link name="odom">
-      <inertial>
-				<mass value="1" />
-				<origin xyz="0.0 0.0 0.0" rpy="0 0 0" />
-				<inertia ixx="0.1" ixy="0.0" ixz="0.0"	iyy="0.1" iyz="0.0" izz="0.1" />
-			</inertial>
-    </link>
-    <joint name="base_x_joint" type="prismatic">
-			<origin xyz="0 0 0" rpy="0 0 0" />
-			<axis xyz="1 0 0"/>
-      <calibration rising="0.0"/>
-      <dynamics damping="0.0" friction="0.0" />
-      <limit effort="10" velocity="1.0" lower="-100" upper="100" />
-			<parent link="odom"/>
-			<child link="base_x_link" />
-		</joint>
-    <link name="base_x_link">
-      <inertial>
-				<mass value="1" />
-				<origin xyz="0 0 0.0" />
-				<inertia ixx="0.1" ixy="0.0" ixz="0.0"	iyy="0.1" iyz="0.0" izz="0.1" />
-			</inertial>
-    </link>
-    <joint name="base_y_joint" type="prismatic">
-			<origin xyz="0 0 0" rpy="0 0 0" />
-			<axis xyz="0 1 0"/>
-      <calibration rising="0.0"/>
-      <dynamics damping="0.0" friction="0.0" />
-      <limit effort="10" velocity="1.0" lower="-100" upper="100" />
-			<parent link="base_x_link"/>
-			<child link="base_y_link" />
-		</joint>
-    <link name="base_y_link">
-      <inertial>
-				<mass value="1" />
-				<origin xyz="0.0 0.0 0.0" rpy="0 0 0" />
-				<inertia ixx="0.1" ixy="0.0" ixz="0.0"	iyy="0.1" iyz="0.0" izz="0.1" />
-        </inertial>
-    </link>
-		<joint name="base_yaw_joint" type="continuous">
-			<origin xyz="0 0 0" rpy="0 0 0" />
-			<axis xyz="0 0 1"/>
-      <calibration rising="0.0"/>
-      <dynamics damping="0.0" friction="0.0" />
-      <limit effort="10" velocity="1.0"/>
-			<parent link="base_y_link"/>
-			<child link="base_link" />
-		</joint>
-		<link name="base_link">
-			<inertial>
-				<mass value="1.0" />
-				<origin xyz="0.0 0.0 0.0" rpy="0 0 0" />
-				<inertia ixx="0.1" ixy="0.0" ixz="0.0"	iyy="0.1" iyz="0.0" izz="0.1" />
-			</inertial>
-      <!-- z verschiebung = Abstand von Boden zu Motor achse + Rad Radius -->
-			<visual>
-				<origin xyz="0 0 ${0.090+0.254/2}" rpy="1.57079 0 1.57079" />
-				<geometry>
-					<mesh filename="package://omnirob_robin_description/meshes/omnirob_base.stl" scale="0.001 0.001 0.001"/>
-				</geometry>
-        <material name="Green">
-          <color rgba="0.5 0.5 0.5 1.0"/>
-        </material>
-			</visual>
-			<collision>
-				<origin xyz="0.0 0.0 0.36" rpy="0 0 0" />
-				<geometry>
-					<cylinder length="0.71" radius="0.425"/>
-				</geometry>
-			</collision>
-		</link>
-    <joint name="base_mass_joint" type="fixed">
-			<origin xyz="0 0 0.4" rpy="0 0 0" />
-			<parent link="base_link"/>
-			<child link="base_mass_link" />
-		</joint>
-    <link name="base_mass_link">
-			<inertial>
-				<mass value="80.0" />
-				<origin xyz="0.0 0.0 0.0" rpy="0 0 0" />
-				<inertia ixx="0.5" ixy="0.0" ixz="0.0"	iyy="0.5" iyz="0.0" izz="0.5" />
-			</inertial>
-		</link>
-		<xacro:if value="${simulated}">
-      <xacro:omnirob_transmission/>
-    </xacro:if>
-	</xacro:macro>
+   <xacro:macro name="base" params="">
+      <link name="world" />
+      <joint name="odom_joint" type="fixed">
+         <parent link="world" />
+         <child link="odom" />
+      </joint>
+      <link name="odom">
+         <inertial>
+            <mass value="1" />
+            <origin xyz="0.0 0.0 0.0" rpy="0 0 0" />
+            <inertia ixx="0.1" ixy="0.0" ixz="0.0" iyy="0.1" iyz="0.0" izz="0.1" />
+         </inertial>
+      </link>
+      <joint name="base_x_joint" type="prismatic">
+         <origin xyz="0 0 0" rpy="0 0 0" />
+         <axis xyz="1 0 0" />
+         <dynamics damping="0.0" friction="0.0" />
+         <limit effort="10" velocity="1.0" lower="-100" upper="100" />
+         <parent link="odom" />
+         <child link="base_x_link" />
+      </joint>
+      <link name="base_x_link">
+         <inertial>
+            <mass value="1" />
+            <origin xyz="0 0 0.0" />
+            <inertia ixx="0.1" ixy="0.0" ixz="0.0" iyy="0.1" iyz="0.0" izz="0.1" />
+         </inertial>
+      </link>
+      <joint name="base_y_joint" type="prismatic">
+         <origin xyz="0 0 0" rpy="0 0 0" />
+         <axis xyz="0 1 0" />
+         <dynamics damping="0.0" friction="0.0" />
+         <limit effort="10" velocity="1.0" lower="-100" upper="100" />
+         <parent link="base_x_link" />
+         <child link="base_y_link" />
+      </joint>
+      <link name="base_y_link">
+         <inertial>
+            <mass value="1" />
+            <origin xyz="0.0 0.0 0.0" rpy="0 0 0" />
+            <inertia ixx="0.1" ixy="0.0" ixz="0.0" iyy="0.1" iyz="0.0" izz="0.1" />
+         </inertial>
+      </link>
+      <joint name="base_yaw_joint" type="continuous">
+         <origin xyz="0 0 0" rpy="0 0 0" />
+         <axis xyz="0 0 1" />
+         <dynamics damping="0.0" friction="0.0" />
+         <limit effort="10" velocity="1.0" lower="-100" upper="100"/>
+         <parent link="base_y_link" />
+         <child link="base_link" />
+      </joint>
+      <link name="base_link">
+         <inertial>
+            <mass value="1.0" />
+            <origin xyz="0.0 0.0 0.0" rpy="0 0 0" />
+            <inertia ixx="0.1" ixy="0.0" ixz="0.0" iyy="0.1" iyz="0.0" izz="0.1" />
+         </inertial>
+         <!-- z verschiebung = Abstand von Boden zu Motor achse + Rad Radius -->
+         <visual>
+            <origin xyz="0 0 ${0.090+0.254/2}" rpy="1.57079 0 1.57079" />
+            <geometry>
+               <mesh filename="package://omnirob_robin_description/meshes/omnirob_base.stl" scale="0.001 0.001 0.001" />
+            </geometry>
+            <material name="Green">
+               <color rgba="0.5 0.5 0.5 1.0" />
+            </material>
+         </visual>
+         <collision>
+            <origin xyz="0.0 0.0 0.36" rpy="0 0 0" />
+            <geometry>
+               <cylinder length="0.71" radius="0.425" />
+            </geometry>
+         </collision>
+      </link>
+      <joint name="base_mass_joint" type="fixed">
+         <origin xyz="0 0 0.4" rpy="0 0 0" />
+         <parent link="base_link" />
+         <child link="base_mass_link" />
+      </joint>
+      <link name="base_mass_link">
+         <inertial>
+            <mass value="80.0" />
+            <origin xyz="0.0 0.0 0.0" rpy="0 0 0" />
+            <inertia ixx="0.5" ixy="0.0" ixz="0.0" iyy="0.5" iyz="0.0" izz="0.5" />
+         </inertial>
+      </link>
+      <xacro:if value="${simulated}">
+		 <xacro:include filename="$(find omnirob_robin_description)/urdf/omnirob_robin_base/base.transmission.xacro" />
+         <xacro:omnirob_transmission />
+      </xacro:if>
+   </xacro:macro>
 </robot>

File: omnirob_robin_description/urdf/schunk_pan_tilt/schunk_pan_tilt.urdf.xacro (robot description, xacro)
@@ -7,5 +7,5 @@
 			<axis xyz="0 0 1"/>
 			<parent link="${parent}"/>
-      <calibration rising="0.0"/>
+      <calibration rising="0.0" falling="0.0"/>
       <dynamics damping="0.2" friction="10.0" />
       <limit effort="10" velocity="0.5" lower="-2.0" upper="2.0"/>
@@ -36,5 +36,5 @@
 			<origin xyz="0 0 0.0951" rpy="0 0 0" />
 			<axis xyz="0 1 0"/>
-      <calibration rising="0.0"/>
+      <calibration rising="0.0" falling="0.0"/>
       <dynamics damping="0.2" friction="10.0" />
       <limit effort="10" velocity="0.5" lower="-1.57" upper="1.57"/>

Commit message: update of robot description to match new pan tilt and base

File: omnirob_robin_description/robots/omnirob.urdf.xacro (robot description, xacro)
@@ -8,8 +8,4 @@
     <insert_block name="camera_mast_origin" />
   </xacro:camera_mast>
-  <xacro:schunk_pan_tilt parent="camera_mast_origin_link">
-    <!-- set in properties xacro -->
-    <insert_block name="pan_tilt_origin" />
-  </xacro:schunk_pan_tilt>
   <xacro:ultrasound_sensor parent="base_link" number="0">
     <insert_block name="ultrasound_sensor0" />
@@ -38,4 +34,7 @@
   <xacro:sensor_kinect parent="pan_tilt/tcp_link" />
   <xacro:sensor_sick3000 parent="base_link" />
+  <xacro:schunk_pan_tilt parent="camera_mast_origin_link">
+    <insert_block name="pan_tilt_origin" />
+  </xacro:schunk_pan_tilt>
   <xacro:lwa parent="base_link" name="lwa">
 	  <insert_block name="lwa_origin"/>

File: omnirob_robin_description/urdf/omnirob_robin.library.xacro (robot description, xacro)
@@ -18,6 +18,7 @@
   <!-- Schunk Pan Tilt
   <xacro:include filename="$(find omnirob_robin_description)/urdf/schunk_pan_tilt/schunk_pan_tilt.urdf.xacro"/>
-   -->
-  <xacro:include filename="$(find omnirob_robin_description)/urdf/power_cube_pan_tilt/power_cube_pan_tilt.urdf.xacro"/>
+  -->
+  <!-- -->
+  <xacro:include filename="$(find omnirob_robin_description)/urdf/power_cube_pan_tilt/schunk_pan_tilt.urdf.xacro"/>
   <!-- lwa -->
   <xacro:include filename="$(find omnirob_robin_description)/urdf/lwa/lwa.urdf.xacro"/>

File: omnirob_robin_description/urdf/omnirob_robin.properties.xacro (robot description, xacro)
@@ -10,5 +10,5 @@
   <xacro:property name="pan_tilt_origin">
     <!-- von camera mast origin zu pan_tilt_origin -->
-    <origin xyz="0 0 0.669" rpy="0 0 0"/>
+    <origin xyz="0 0 0.54" rpy="0 0 0"/>
   </xacro:property>
   <property name="arm_1_ref" value="0"/>
@@ -41,5 +41,5 @@
     <origin xyz="${0.7/2.0+0.003+0.0597} 0 ${0.293+0.116}" rpy="${M_PI} 0 0"/>
   </xacro:property>
-  <property name="ultrasound_z" value="0.66"/>
+  <property name="ultrasound_z" value="0.655"/>
   <property name="ultrasound_offset" value="0.34"/>
   <property name="sqrt2" value="1.414213562"/>

File: omnirob_robin_description/urdf/omnirob_robin_base/base.urdf.xacro (robot description, xacro)
@@ -62,5 +62,5 @@
             <origin xyz="0 0 0" rpy="1.57079 0 1.57079" />
             <geometry>
-               <mesh filename="package://omnirob_robin_description/meshes/omnirob.stl" scale="0.001 0.001 0.001" />
+               <mesh filename="package://omnirob_robin_description/meshes/omnirob.dae" scale="0.001 0.001 0.001" />
             </geometry>
             <material name="Green">

File: omnirob_robin_description/urdf/power_cube_pan_tilt/schunk_pan_tilt.urdf.xacro (robot description, xacro)
@@ -1,82 +1,104 @@
-<?xml version="1.0"?>
+<?xml version="1.0" encoding="UTF-8"?>
 <robot xmlns:xacro="http://ros.org/wiki/xacro">
-	<xacro:include filename="$(find omnirob_robin_description)/urdf/schunk_pan_tilt/schunk_pan_tilt.transmission.xacro"/>
-	<xacro:macro name="schunk_pan_tilt" params="parent *origin">
+   <xacro:include filename="$(find omnirob_robin_description)/urdf/schunk_pan_tilt/schunk_pan_tilt.transmission.xacro" />
+   <xacro:macro name="schunk_pan_tilt" params="parent *origin">
+      <joint name="pan_tilt/pan_socket_joint" type="fixed">
+         <insert_block name="origin" />
+         <parent link="${parent}" />
+         <child link="pan_tilt/pan_socket_link" />
+      </joint>
+      <link name="pan_tilt/pan_socket_link">
+         <inertial>
+            <mass value="0.5" />
+            <origin xyz="0 0 0.0" />
+            <inertia ixx="0.01" ixy="0.0" ixz="0.0" iyy="0.01" iyz="0.0" izz="0.5" />
+         </inertial>
+         <visual>
+            <origin xyz="0 0 0" rpy="0 0 0" />
+            <geometry>
+               <mesh filename="package://omnirob_robin_description/meshes/power_cube_pan_socket.stl" scale="0.001 0.001 0.001" />
+            </geometry>
+            <material name="Schunk/DarkGolden" />
+         </visual>
+         <collision>
+            <origin xyz="0.0 0.0 0.05" rpy="0 0 0" />
+            <geometry>
+               <box size="0.1 0.1 0.1" />
+            </geometry>
+         </collision>
+      </link>
     <joint name="pan_tilt/pan_joint" type="continuous">
-			<insert_block name="origin"/>
-			<axis xyz="0 0 1"/>
-			<parent link="${parent}"/>
-      <calibration rising="0.0" falling="0.0"/>
-      <dynamics damping="0.2" friction="10.0" />
-      <limit effort="10" velocity="0.5" lower="-2.0" upper="2.0"/>
-			<child link="pan_tilt/pan_link" />
-		</joint>
-		<link name="pan_tilt/pan_link">
-			<inertial>
-				<mass value="0.5" />
-				<origin xyz="0 0 0.0" />
-				<inertia ixx="0.01" ixy="0.0" ixz="0.0"
-					iyy="0.01" iyz="0.0" izz="0.5" />
-			</inertial>
-      <visual>
-				<origin xyz="0 0 0.094" rpy="0 ${M_PI} ${M_PI/2}" />
-				<geometry>
-					<mesh filename="package://omnirob_robin_description/meshes/power_cube_pan.stl" scale="0.001 0.001 0.001"/>
-				</geometry>
-        <material name="Schunk/DarkGolden" />
-			</visual>
-      <collision>
-				<origin xyz="0.0 0.0 0.08" rpy="0 0 0" />
-				<geometry>
-					<box size="0.1 0.12 0.16"/>
-				</geometry>
-			</collision>
-		</link>
-    <joint name="pan_tilt/tilt_joint" type="continuous">
-			<origin xyz="0 0 0.0951" rpy="0 0 0" />
-			<axis xyz="0 1 0"/>
-      <calibration rising="0.0" falling="0.0"/>
-      <dynamics damping="0.2" friction="10.0" />
-      <limit effort="10" velocity="0.5" lower="-1.57" upper="1.57"/>
-			<parent link="pan_tilt/pan_link"/>
-			<child link="pan_tilt/tilt_link" />
-		</joint>
-		<link name="pan_tilt/tilt_link">
-			<inertial>
-				<mass value="0.5" />
-				<origin xyz="0 0 0.0" />
-				<inertia ixx="0.01" ixy="0.0" ixz="0.0"
-					iyy="0.01" iyz="0.0" izz="0.5" />
-			</inertial>
-      <visual>
-				<origin xyz=" 0 0 0" rpy="0 ${M_PI} -${M_PI/2}" />
-				<geometry>
-					<mesh filename="package://omnirob_robin_description/meshes/schunk_tilt.stl" scale="0.001 0.001 0.001"/>
-				</geometry>
-        <material name="Schunk/DarkGolden" />
-			</visual>
-      <collision>
-				<origin xyz="0.0 0.0 0.0" rpy="0 0 0" />
-				<geometry>
-					<box size="0.12 0.24 0.11"/>
-				</geometry>
-			</collision>
-		</link>
-     <joint name="pan_tilt/tcp_joint" type="fixed">
-			<origin xyz="0 0 0.07" rpy="0 0 0" />
-			<parent link="pan_tilt/tilt_link"/>
-			<child link="pan_tilt/tcp_link" />
-		</joint>
-		<link name="pan_tilt/tcp_link">
-			<inertial>
-				<mass value="0.5" />
-				<origin xyz="0 0 0.0" />
-				<inertia ixx="0.01" ixy="0.0" ixz="0.0"
-					iyy="0.01" iyz="0.0" izz="0.5" />
-			</inertial>
-		</link>
-    <xacro:if value="${simulated}">
-      <xacro:pan_tilt_transmission/>
-    </xacro:if>
-	</xacro:macro>
+         <origin xyz="0 0 ${0.045+0.071}" rpy="0 0 0" />
+         <axis xyz="0 0 1" />
+         <parent link="pan_tilt/pan_socket_link" />
+         <calibration rising="0.0" falling="0.0" />
+         <dynamics damping="0.2" friction="10.0" />
+         <limit effort="10" velocity="0.5" lower="-2.0" upper="2.0" />
+         <child link="pan_tilt/pan_link" />
+      </joint>
+      <link name="pan_tilt/pan_link">
+         <inertial>
+            <mass value="0.5" />
+            <origin xyz="0 0 0.0" />
+            <inertia ixx="0.01" ixy="0.0" ixz="0.0" iyy="0.01" iyz="0.0" izz="0.5" />
+         </inertial>
+         <visual>
+            <origin xyz="0 0 0" rpy="0 0 ${M_PI/2.0}" />
+            <geometry>
+               <mesh filename="package://omnirob_robin_description/meshes/power_cube_pan.stl" scale="0.001 0.001 0.001" />
+            </geometry>
+            <material name="Schunk/DarkGolden" />
+         </visual>
+         <collision>
+            <origin xyz="0.0 0.0 0.08" rpy="0 0 0" />
+            <geometry>
+               <box size="0.1 0.12 0.16" />
+            </geometry>
+         </collision>
+      </link>
+      <joint name="pan_tilt/tilt_joint" type="continous">
+         <origin xyz="0 ${-0.071/2} ${0.071+0.04+0.071/2}" rpy="0 0 0" />
+         <axis xyz="0 1 0" />
+         <calibration rising="0.0" falling="0.0" />
+         <dynamics damping="0.2" friction="10.0" />
+         <limit effort="10" velocity="0.5" lower="-1.57" upper="1.57" />
+         <parent link="pan_tilt/pan_link" />
+         <child link="pan_tilt/tilt_link" />
+      </joint>
+      <link name="pan_tilt/tilt_link">
+         <inertial>
+            <mass value="0.5" />
+            <origin xyz="0 0 0.0" />
+            <inertia ixx="0.01" ixy="0.0" ixz="0.0" iyy="0.01" iyz="0.0" izz="0.5" />
+         </inertial>
+         <visual>
+            <origin xyz=" 0 0 0" rpy="0 0 0" />
+            <geometry>
+               <mesh filename="package://omnirob_robin_description/meshes/power_cube_tilt.stl" scale="0.001 0.001 0.001" />
+            </geometry>
+            <material name="Schunk/DarkGolden" />
+         </visual>
+         <collision>
+            <origin xyz="0.0 0.0 0.0" rpy="0 0 0" />
+            <geometry>
+               <box size="0.12 0.24 0.11" />
+            </geometry>
+         </collision>
+      </link>
+      <joint name="pan_tilt/tcp_joint" type="fixed">
+         <origin xyz="0 0 0.07" rpy="0 0 0" />
+         <parent link="pan_tilt/tilt_link" />
+         <child link="pan_tilt/tcp_link" />
+      </joint>
+      <link name="pan_tilt/tcp_link">
+         <inertial>
+            <mass value="0.5" />
+            <origin xyz="0 0 0.0" />
+            <inertia ixx="0.01" ixy="0.0" ixz="0.0" iyy="0.01" iyz="0.0" izz="0.5" />
+         </inertial>
+      </link>
+      <xacro:if value="${simulated}">
+         <xacro:pan_tilt_transmission />
+      </xacro:if>
+   </xacro:macro>
 </robot>

File: omnirob_robin_description/urdf/sensors/Ultrasound.urdf.xacro (robot description, xacro)
@@ -20,7 +20,7 @@
 					<box size="0.02 0.05 0.02" />
 				</geometry>
-        <material name="Green">
-          <color rgba="0.0 0.0 0.0 1.0"/>
-        </material>
+                <material name="yellow">
+                    <color rgba="1.0 1.0 0 1"/>
+                </material>
 			</visual>
 			<collision>

File: omnirob_robin_description/urdf/sensors/sick3000.urdf.xacro (robot description, xacro)
@@ -24,4 +24,7 @@
           <box size="0.106 0.102 0.152"/>
         </geometry>
+        <material name="yellow">
+            <color rgba="1.0 1.0 0 1"/>
+        </material>
       </visual>
       <collision>
