Commit message: Real and simulated interfaces launch files fixed

File: omnirob_robin_description/robots/omnirob_robin_real.urdf.xacro (robot description, xacro)
@@ -2,4 +2,7 @@
 <robot name="omnirob_robin" xmlns:xacro="http://ros.org/wiki/xacro">
   <xacro:property name="simulated" value="0" />
+  <xacro:property name="ofx" value="0" />
+  <xacro:property name="ofx" value="0" />
+  <xacro:property name="ofx" value="0" />
   <xacro:include filename="$(find omnirob_robin_description)/robots/omnirob.urdf.xacro" />
 </robot>

File: omnirob_robin_description/urdf/omnirob_robin_base/base.urdf.xacro (robot description, xacro)
@@ -5,5 +5,7 @@
       <link name="world" />
       <joint name="odom_joint" type="fixed">
-		 <origin xyz="$(arg ofx) $(arg ofy) $(arg ofz)" rpy="0 0 0" />
+         <xacro:if value="${simulated}">
+            <origin xyz="$(arg ofx) $(arg ofy) $(arg ofz)" rpy="0 0 0" />
+         </xacro:if>
          <parent link="world" />
          <child link="odom" />
