Commit message: Ultraschallsensoren links in urdf Dateien geändert

File: omnirob_robin_description/urdf/sensors/Ultrasound.urdf.xacro (robot description, xacro)
@@ -5,7 +5,7 @@
 			<insert_block name="origin" />
 			<parent link="${parent}" />
-			<child link="ultrasound_sensor${number}_origin_link" />
+			<child link="US${number}_link" />
 		</joint>
-		<link name="ultrasound_sensor${number}_origin_link">
+		<link name="US${number}_link">
 			<inertial>
 				<mass value="0.1" />
