Commit message: object_detection adapted to pan_tilt_interface, gripper velocity limits set

File: omnirob_robin_description/urdf/pg70/pg70.urdf.xacro (robot description, xacro)
@@ -42,5 +42,5 @@
       <parent link="${name}/palm_link" />
       <child link="${name}/finger_left_link" />
-      <limit effort="500" lower="0.0" upper="0.035" velocity="2.0"/>
+      <limit effort="10" lower="0.0" upper="0.035" velocity="0.5"/>
       <origin xyz="0 0.005 ${0.078+0.09}" rpy="0 0 0"/>
       <axis xyz="0 1 0" />
@@ -77,5 +77,5 @@
       <parent link="${name}/palm_link" />
       <child link="${name}/finger_right_link" />
-      <limit effort="500" lower="0.0" upper="0.035" velocity="2.0"/>
+      <limit effort="10" lower="0.0" upper="0.035" velocity="0.5"/>
       <origin xyz="0 -0.005 ${0.078+0.09}" rpy="0 0 0"/>
       <axis xyz="0 -1 0" />

Commit message: updated limites for gripper and pan tilt unit

File: omnirob_robin_description/urdf/pg70/pg70.urdf.xacro (robot description, xacro)
@@ -42,5 +42,5 @@
       <parent link="${name}/palm_link" />
       <child link="${name}/finger_left_link" />
-      <limit effort="10" lower="0.0" upper="0.035" velocity="0.5"/>
+      <limit effort="10" lower="0.005" upper="0.025" velocity="0.5"/>
       <origin xyz="0 0.005 ${0.078+0.09}" rpy="0 0 0"/>
       <axis xyz="0 1 0" />
@@ -77,5 +77,5 @@
       <parent link="${name}/palm_link" />
       <child link="${name}/finger_right_link" />
-      <limit effort="10" lower="0.0" upper="0.035" velocity="0.5"/>
+      <limit effort="10" lower="0.005" upper="0.025" velocity="0.5"/>
       <origin xyz="0 -0.005 ${0.078+0.09}" rpy="0 0 0"/>
       <axis xyz="0 -1 0" />

File: omnirob_robin_description/urdf/schunk_pan_tilt/schunk_pan_tilt.urdf.xacro (robot description, xacro)
@@ -9,5 +9,5 @@
       <calibration rising="0.0"/>
       <dynamics damping="0.2" friction="10.0" />
-      <limit effort="10" velocity="0.5"/>
+      <limit effort="10" velocity="0.5" lower="-2.0" upper="2.0"/>
 			<child link="pan_tilt/pan_link" />
 		</joint>
@@ -38,5 +38,5 @@
       <calibration rising="0.0"/>
       <dynamics damping="0.2" friction="10.0" />
-      <limit effort="10" velocity="0.5"/>
+      <limit effort="10" velocity="0.5" lower="-1.57" upper="1.57"/>
 			<parent link="pan_tilt/pan_link"/>
 			<child link="pan_tilt/tilt_link" />
