Commit message: Kinect 2 and Schunk Pan tilt collision boxes enlarged

File: omnirob_robin_description/urdf/schunk_pan_tilt/schunk_pan_tilt.urdf.xacro (robot description, xacro)
@@ -27,7 +27,7 @@
 			</visual>
       <collision>
-				<origin xyz="0.0 0.0 0.07" rpy="0 0 0" />
+				<origin xyz="0.0 0.0 0.08" rpy="0 0 0" />
 				<geometry>
-					<box size="0.07 0.09 0.14"/>
+					<box size="0.08 0.1 0.16"/>
 				</geometry>
 			</collision>
@@ -57,7 +57,7 @@
 			</visual>
       <collision>
-				<origin xyz="0.0 0.018 0.015" rpy="0 0 0" />
+				<origin xyz="0.0 0.0 0.0" rpy="0 0 0" />
 				<geometry>
-					<box size="0.07 0.18 0.1"/>
+					<box size="0.08 0.2 0.11"/>
 				</geometry>
 			</collision>

File: omnirob_robin_description/urdf/sensors/kinect2.urdf.xacro (robot description, xacro)
@@ -23,7 +23,7 @@
     </visual>
 	  <collision>
-      <origin xyz="0.0 0.0 ${0.067/2.0}" rpy="0 0 0"/>
+      <origin xyz="0.0 0.0 ${0.08/2.0}" rpy="0 0 0"/>
 	    <geometry>
-	      <box size="0.066 0.249 0.067"/>
+	      <box size="0.08 0.260 0.08"/>
 	    </geometry>
 	  </collision>

Commit message: kinect and schunk pan tilt collision boxes enlarged

File: omnirob_robin_description/urdf/schunk_pan_tilt/schunk_pan_tilt.urdf.xacro (robot description, xacro)
@@ -29,5 +29,5 @@
 				<origin xyz="0.0 0.0 0.08" rpy="0 0 0" />
 				<geometry>
-					<box size="0.08 0.1 0.16"/>
+					<box size="0.1 0.12 0.16"/>
 				</geometry>
 			</collision>
@@ -59,5 +59,5 @@
 				<origin xyz="0.0 0.0 0.0" rpy="0 0 0" />
 				<geometry>
-					<box size="0.08 0.2 0.11"/>
+					<box size="0.12 0.24 0.11"/>
 				</geometry>
 			</collision>

File: omnirob_robin_description/urdf/sensors/kinect2.urdf.xacro (robot description, xacro)
@@ -23,7 +23,7 @@
     </visual>
 	  <collision>
-      <origin xyz="0.0 0.0 ${0.08/2.0}" rpy="0 0 0"/>
+      <origin xyz="0.0 0.0 ${0.1/2.0}" rpy="0 0 0"/>
 	    <geometry>
-	      <box size="0.08 0.260 0.08"/>
+	      <box size="0.12 0.35 0.12"/>
 	    </geometry>
 	  </collision>
