Commit message: joint limits for new pan tilt unit

File: omnirob_robin_description/urdf/power_cube_pan_tilt/schunk_pan_tilt.urdf.xacro (robot description, xacro)
@@ -57,5 +57,5 @@
          </collision>
       </link>
-      <joint name="pan_tilt/tilt_joint" type="continous">
+      <joint name="pan_tilt/tilt_joint" type="continuous">
          <origin xyz="0 ${-0.071/2} ${0.071+0.04+0.071/2}" rpy="0 0 0" />
          <axis xyz="0 1 0" />
