Commit message: added interfaces to real launch, fixed some joint names for tf

File: omnirob_robin_description/urdf/omnirob_robin_base/base.transmission.xacro (robot description, xacro)
@@ -4,5 +4,5 @@
     <transmission name="tran_x">
         <type>transmission_interface/SimpleTransmission</type>
-        <joint name="base/x_joint">
+        <joint name="base_x_joint">
           <hardwareInterface>PositionJointInterface</hardwareInterface>
         </joint>
@@ -14,5 +14,5 @@
     <transmission name="tran_y">
         <type>transmission_interface/SimpleTransmission</type>
-        <joint name="base/y_joint">
+        <joint name="base_y_joint">
           <hardwareInterface>PositionJointInterface</hardwareInterface>
         </joint>
@@ -24,5 +24,5 @@
     <transmission name="tran_yaw">
         <type>transmission_interface/SimpleTransmission</type>
-        <joint name="base/yaw_joint">
+        <joint name="base_yaw_joint">
           <hardwareInterface>PositionJointInterface</hardwareInterface>
         </joint>

File: omnirob_robin_description/urdf/omnirob_robin_base/base.urdf.xacro (robot description, xacro)
@@ -16,5 +16,5 @@
 			</inertial>
     </link>
-    <joint name="base/x_joint" type="prismatic">
+    <joint name="base_x_joint" type="prismatic">
 			<origin xyz="0 0 0" rpy="0 0 0" />
 			<axis xyz="1 0 0"/>
@@ -23,7 +23,7 @@
       <limit effort="10" velocity="1.0" lower="-100" upper="100" />
 			<parent link="odom"/>
-			<child link="base/x_link" />
+			<child link="base_x_link" />
 		</joint>
-    <link name="base/x_link">
+    <link name="base_x_link">
       <inertial>
 				<mass value="1" />
@@ -32,5 +32,5 @@
 			</inertial>
     </link>
-    <joint name="base/y_joint" type="prismatic">
+    <joint name="base_y_joint" type="prismatic">
 			<origin xyz="0 0 0" rpy="0 0 0" />
 			<axis xyz="0 1 0"/>
@@ -38,8 +38,8 @@
       <dynamics damping="0.0" friction="0.0" />
       <limit effort="10" velocity="1.0" lower="-100" upper="100" />
-			<parent link="base/x_link"/>
-			<child link="base/y_link" />
+			<parent link="base_x_link"/>
+			<child link="base_y_link" />
 		</joint>
-    <link name="base/y_link">
+    <link name="base_y_link">
       <inertial>
 				<mass value="1" />
@@ -48,5 +48,5 @@
         </inertial>
     </link>
-		<joint name="base/yaw_joint" type="continuous">
+		<joint name="base_yaw_joint" type="continuous">
 			<origin xyz="0 0 0" rpy="0 0 0" />
 			<axis xyz="0 0 1"/>
@@ -54,5 +54,5 @@
       <dynamics damping="0.0" friction="0.0" />
       <limit effort="10" velocity="1.0"/>
-			<parent link="base/y_link"/>
+			<parent link="base_y_link"/>
 			<child link="base_link" />
 		</joint>
@@ -80,10 +80,10 @@
 			</collision>
 		</link>
-    <joint name="base/mass_joint" type="fixed">
+    <joint name="base_mass_joint" type="fixed">
 			<origin xyz="0 0 0.4" rpy="0 0 0" />
 			<parent link="base_link"/>
-			<child link="base/mass_link" />
+			<child link="base_mass_link" />
 		</joint>
-    <link name="base/mass_link">
+    <link name="base_mass_link">
 			<inertial>
 				<mass value="80.0" />

Commit message: URDF fixes

File: omnirob_robin_description/urdf/omnirob_robin_base/base.transmission.xacro (robot description, xacro)
@@ -8,6 +8,6 @@
         </joint>
         <actuator name="motor_x">
+		  <mechanicalReduction>1</mechanicalReduction>
           <hardwareInterface>PositionJointInterface</hardwareInterface>
-          <mechanicalReduction>1</mechanicalReduction>
         </actuator>
     </transmission>

File: omnirob_robin_description/urdf/omnirob_robin_base/base.urdf.xacro (robot description, xacro)
@@ -1,4 +1,5 @@
 <?xml version="1.0" encoding="UTF-8"?>
 <robot xmlns:xacro="http://ros.org/wiki/xacro">
+   <xacro:include filename="$(find omnirob_robin_description)/urdf/omnirob_robin_base/base.transmission.xacro" />
    <xacro:macro name="base" params="">
       <link name="world" />
@@ -18,4 +19,5 @@
          <axis xyz="1 0 0" />
          <dynamics damping="0.0" friction="0.0" />
+         <calibration rising="0.0" falling="0.0" />
          <limit effort="10" velocity="1.0" lower="-100" upper="100" />
          <parent link="odom" />
@@ -88,5 +90,4 @@
       </link>
       <xacro:if value="${simulated}">
-		 <xacro:include filename="$(find omnirob_robin_description)/urdf/omnirob_robin_base/base.transmission.xacro" />
          <xacro:omnirob_transmission />
       </xacro:if>

File: omnirob_robin_description/urdf/sensors/Ultrasound.urdf.xacro (robot description, xacro)
@@ -11,8 +11,6 @@
 				<mass value="0.1" />
 				<origin xyz="0 0.0 0.0" />
-			an_tilt_origin	<inertia ixx="0.0" ixy="0.0" ixz="0.0"
-					iyy="0.0" iyz="0.0" izz="0.0" />
+				<inertia ixx="0.0" ixy="0.0" ixz="0.0"	iyy="0.0" iyz="0.0" izz="0.0" />
 			</inertial>
-      <!-- sensor-origin is the center of the vertical post -->
 			<visual>
 				<origin xyz="0 0 0" rpy="0 0 0" />
