Commit message: Fixed tf tree in simulation

File: omnirob_robin_description/urdf/omnirob_robin_base/base.urdf.xacro (robot description, xacro)
@@ -5,4 +5,15 @@
 	<xacro:macro name="base" params="">
     <link name="world" />
+    <joint name="odom_joint" type="fixed">
+			<parent link="world"/>
+			<child link="odom" />
+		</joint>
+    <link name="odom">
+      <inertial>
+				<mass value="1" />
+				<origin xyz="0 0 0.0" />
+				<inertia ixx="0.1" ixy="0.0" ixz="0.0"	iyy="0.1" iyz="0.0" izz="0.1" />
+			</inertial>
+    </link>
     <joint name="base/x_joint" type="prismatic">
 			<origin xyz="0 0 0" rpy="0 0 0" />
@@ -11,5 +22,5 @@
       <dynamics damping="0.0" friction="0.0" />
       <limit effort="10" velocity="1.0" lower="-100" upper="100" />
-			<parent link="world"/>
+			<parent link="odom"/>
 			<child link="base/x_link" />
 		</joint>

Commit message: fixed urdf for web visualization

File: omnirob_robin_description/urdf/omnirob_robin_base/base.urdf.xacro (robot description, xacro)
@@ -12,5 +12,5 @@
       <inertial>
 				<mass value="1" />
-				<origin xyz="0 0 0.0" />
+				<origin xyz="0.0 0.0 0.0" rpy="0 0 0" />
 				<inertia ixx="0.1" ixy="0.0" ixz="0.0"	iyy="0.1" iyz="0.0" izz="0.1" />
 			</inertial>
@@ -44,5 +44,5 @@
       <inertial>
 				<mass value="1" />
-				<origin xyz="0 0 0.0" />
+				<origin xyz="0.0 0.0 0.0" rpy="0 0 0" />
 				<inertia ixx="0.1" ixy="0.0" ixz="0.0"	iyy="0.1" iyz="0.0" izz="0.1" />
         </inertial>
@@ -60,10 +60,10 @@
 			<inertial>
 				<mass value="1.0" />
-				<origin xyz="0 0 0" />
+				<origin xyz="0.0 0.0 0.0" rpy="0 0 0" />
 				<inertia ixx="0.1" ixy="0.0" ixz="0.0"	iyy="0.1" iyz="0.0" izz="0.1" />
 			</inertial>
       <!-- z verschiebung = Abstand von Boden zu Motor achse + Rad Radius -->
 			<visual>
-				<origin xyz=" 0 0 ${0.090+0.254/2}" rpy="1.57079 0 1.57079" />
+				<origin xyz="0 0 ${0.090+0.254/2}" rpy="1.57079 0 1.57079" />
 				<geometry>
 					<mesh filename="package://omnirob_robin_description/meshes/omnirob_base.stl" scale="0.001 0.001 0.001"/>
@@ -88,5 +88,5 @@
 			<inertial>
 				<mass value="80.0" />
-				<origin xyz="0 0 0" />
+				<origin xyz="0.0 0.0 0.0" rpy="0 0 0" />
 				<inertia ixx="0.5" ixy="0.0" ixz="0.0"	iyy="0.5" iyz="0.0" izz="0.5" />
 			</inertial>

File: omnirob_robin_description/urdf/schunk_pan_tilt/schunk_pan_tilt.urdf.xacro (robot description, xacro)
@@ -20,5 +20,5 @@
 			</inertial>
       <visual>
-				<origin xyz=" 0 0 0.094" rpy="0 ${M_PI} ${M_PI/2}" />
+				<origin xyz="0 0 0.094" rpy="0 ${M_PI} ${M_PI/2}" />
 				<geometry>
 					<mesh filename="package://omnirob_robin_description/meshes/schunk_pan.stl" scale="0.001 0.001 0.001"/>

Commit message: New version of omnirob visualization model

File: omnirob_robin_description/urdf/omnirob_robin_base/base.urdf.xacro (robot description, xacro)
@@ -60,7 +60,7 @@
          <!-- z verschiebung = Abstand von Boden zu Motor achse + Rad Radius -->
          <visual>
-            <origin xyz="0 0 ${0.090+0.254/2}" rpy="1.57079 0 1.57079" />
+            <origin xyz="0 0 0" rpy="1.57079 0 1.57079" />
             <geometry>
-               <mesh filename="package://omnirob_robin_description/meshes/omnirob_base.stl" scale="0.001 0.001 0.001" />
+               <mesh filename="package://omnirob_robin_description/meshes/omnirob.stl" scale="0.001 0.001 0.001" />
             </geometry>
             <material name="Green">

Commit message: Fixed base visualization

File: omnirob_robin_description/urdf/omnirob_robin_base/base.urdf.xacro (robot description, xacro)
@@ -62,5 +62,5 @@
             <origin xyz="0 0 0" rpy="1.57079 0 1.57079" />
             <geometry>
-               <mesh filename="package://omnirob_robin_description/meshes/omnirob.dae" scale="0.001 0.001 0.001" />
+               <mesh filename="package://omnirob_robin_description/meshes/omnirob.stl" scale="0.001 0.001 0.001" />
             </geometry>
             <material name="Green">

Commit message: Demo changed to Pan_Tilt localization and other improvements

File: omnirob_robin_description/urdf/omnirob_robin_base/base.urdf.xacro (robot description, xacro)
@@ -62,7 +62,7 @@
             <origin xyz="0 0 0" rpy="1.57079 0 1.57079" />
             <geometry>
-               <mesh filename="package://omnirob_robin_description/meshes/omnirob.stl" scale="0.001 0.001 0.001" />
+               <mesh filename="package://omnirob_robin_description/meshes/omnirob.dae" scale="0.001 0.001 0.001" />
             </geometry>
-            <material name="Green">
+            <material name="test">
                <color rgba="0.5 0.5 0.5 1.0" />
             </material>

Commit message: Updated position of the robot in the virtual world. Position is now relative to the world frame instead of moving the world frame.

File: omnirob_robin_description/urdf/omnirob_robin_base/base.urdf.xacro (robot description, xacro)
@@ -5,4 +5,5 @@
       <link name="world" />
       <joint name="odom_joint" type="fixed">
+		 <origin xyz="$(arg ofx) $(arg ofy) $(arg ofz)" rpy="0 0 0" />
          <parent link="world" />
          <child link="odom" />

Commit message: Removed world frame and changed standard localization to amcl

File: omnirob_robin_description/urdf/omnirob_robin_base/base.urdf.xacro (robot description, xacro)
@@ -3,12 +3,4 @@
    <xacro:include filename="$(find omnirob_robin_description)/urdf/omnirob_robin_base/base.transmission.xacro" />
    <xacro:macro name="base" params="">
-      <link name="world" />
-      <joint name="odom_joint" type="fixed">
-         <xacro:if value="${simulated}">
-            <origin xyz="$(arg ofx) $(arg ofy) $(arg ofz)" rpy="0 0 0" />
-         </xacro:if>
-         <parent link="world" />
-         <child link="odom" />
-      </joint>
       <link name="odom">
          <inertial>
