Commit message: fixed gripper orientation in urdf

File: omnirob_robin_description/urdf/omnirob_robin.properties.xacro (robot description, xacro)
@@ -27,5 +27,5 @@
   </xacro:property>
   <xacro:property name="gripper_origin">
-    <origin xyz="0 0 -0.02" rpy="${M_PI} 0 0"/>
+    <origin xyz="0 0 -0.02" rpy="${M_PI} 0 ${M_PI/2.0}"/>
   </xacro:property>
   <!-- camera rgb frame position von pan_tilt_tilt zentrum gemessen -->

Commit message: lwa placement in urdf updated

File: omnirob_robin_description/urdf/omnirob_robin.properties.xacro (robot description, xacro)
@@ -23,6 +23,6 @@
          x = roboterlaenge / 2 - plattenlaenge halbe - versatz
          y = mittig
-         z = raddurchmesser/2 + achsabstand zur unterseite der platform + platformhoehe + profilhoehe -->
-    <origin xyz="${0.7/2-0.355/2-0.094} 0 ${0.254/2+0.09+0.457+0.04}" rpy="${M_PI} 0 0"/>
+         z = raddurchmesser/2 + achsabstand zur unterseite der platform + platformhoehe + profilhoehe + Sockeloffset -->
+    <origin xyz="${0.7/2-0.355/2-0.094} 0 ${0.254/2+0.09+0.457+0.04+0.06}" rpy="${M_PI} 0 0"/>
   </xacro:property>
   <xacro:property name="gripper_origin">

Commit message: Fixed pan_tilt height

File: omnirob_robin_description/urdf/omnirob_robin.properties.xacro (robot description, xacro)
@@ -10,5 +10,5 @@
   <xacro:property name="pan_tilt_origin">
     <!-- von camera mast origin zu pan_tilt_origin -->
-    <origin xyz="0 0 0.54" rpy="0 0 0"/>
+    <origin xyz="0 0 0.484" rpy="0 0 0"/>
   </xacro:property>
   <property name="arm_1_ref" value="0"/>
